Commit message: initial fisheye implementation

File: site/RacingSim/Sensors/av24.urdf (robot description, URDF)
Before this commit: robot AV24, 24 links, 22 joints
Links:
- removed link camera_front_1
- removed link camera_front_2
- removed link camera_rear_left
- removed link camera_rear_right
- removed link gps_bottom_primary_antenna
- removed link gps_bottom_secondary_antenna
- removed link gps_top_primary_antenna
- removed link gps_top_secondary_antenna
- removed link radar_port
- removed link radar_starboard
- removed link vectornav
- removed link vectornav_primary_antenna
- removed link vectornav_secondary_antenna
- added link base_link; visual mesh filename=package://av21_description/models/av21.dae
- added link camera_front_roll_hoop
- added link camera_front_stereo_left
- added link camera_front_stereo_right
- added link camera_rear_roll_hoop
- added link front_axle_middle
- added link gps_bottom_ant1
- added link gps_bottom_imu
- added link gps_spare
- added link gps_spare_imu
- added link gps_top_ant1
- added link gps_top_imu
- added link rear_axle_middle_ground
Joints:
- removed joint camera_front_1_joint
- removed joint camera_front_2_joint
- removed joint camera_front_left_joint
- removed joint camera_front_right_joint
- removed joint camera_rear_left_joint
- removed joint camera_rear_right_joint
- removed joint gps_bottom_joint
- removed joint gps_bottom_primary_antenna_joint
- removed joint gps_bottom_secondary_antenna_joint
- removed joint gps_top_joint
- removed joint gps_top_primary_antenna_joint
- removed joint gps_top_secondary_antenna_joint
- removed joint luminar_front_joint
- removed joint luminar_left_joint
- removed joint luminar_right_joint
- removed joint radar_front_joint
- removed joint radar_port_joint
- removed joint radar_starboard_joint
- removed joint rear_axle_middle_joint
- removed joint vectornav_joint
- removed joint vectornav_primary_antenna_joint
- removed joint vectornav_secondary_antenna_joint
- added joint base_link_to_rear_axle_middle: type fixed, parent base_link, child rear_axle_middle, origin xyz=0.0 0.0 0.0 rpy=0.0 0.0 0.0
- added joint gps_bottom_to_imu_bottom: type fixed, parent gps_bottom, child gps_bottom_imu, origin xyz=0.0 0.0 0.0 rpy=0.0 0.0 -1.5707963267949
- added joint gps_spare_to_imu_spare: type fixed, parent gps_spare, child gps_spare_imu, origin xyz=0.0 0.0 0.0 rpy=0.0 0.0 0.0
- added joint gps_top_to_imu_top: type fixed, parent gps_top, child gps_top_imu, origin xyz=0.0 0.0 0.0 rpy=0.0 0.0 -1.5707963267949
- added joint rear_axle_ground_to_camera_front_left: type fixed, parent rear_axle_middle, child camera_front_left, origin xyz=2.020 0.172 0.418 rpy=0 0 1.745327778
- added joint rear_axle_ground_to_camera_front_right: type fixed, parent rear_axle_middle, child camera_front_right, origin xyz=2.020 -0.172 0.418 rpy=0 0 -1.745327778
- added joint rear_axle_ground_to_camera_front_roll_hoop: type fixed, parent rear_axle_middle, child camera_front_roll_hoop, origin xyz=1.365 0.0 0.723 rpy=0 0 0
- added joint rear_axle_ground_to_camera_rear_roll_hoop: type fixed, parent rear_axle_middle, child camera_rear_roll_hoop, origin xyz=1.215 0.0 0.723 rpy=0 0 3.14159
- added joint rear_axle_ground_to_camera_stereo_left: type fixed, parent rear_axle_middle, child camera_front_stereo_left, origin xyz=2.232 0.180 0.442 rpy=0.0 0.0 0.0
- added joint rear_axle_ground_to_camera_stereo_right: type fixed, parent rear_axle_middle, child camera_front_stereo_right, origin xyz=2.232 -0.180 0.442 rpy=0.0 0.0 0.0
- added joint rear_axle_ground_to_gps_bottom: type fixed, parent rear_axle_middle, child gps_bottom, origin xyz=1.636 0.075 -0.101 rpy=0.0 0.0 0.0
- added joint rear_axle_ground_to_gps_bottom_ant1: type fixed, parent rear_axle_middle, child gps_bottom_ant1, origin xyz=2.055 -0.497 0.353 rpy=0.0 0.0 0.0
- added joint rear_axle_ground_to_gps_spare: type fixed, parent rear_axle_middle, child gps_spare, origin xyz=1.754 0.0 -0.118 rpy=0.0 0.0 0.0
- added joint rear_axle_ground_to_gps_top: type fixed, parent rear_axle_middle, child gps_top, origin xyz=1.636 -0.075 -0.101 rpy=0.0 0.0 0.0
- added joint rear_axle_ground_to_gps_top_ant1: type fixed, parent rear_axle_middle, child gps_top_ant1, origin xyz=3.176 0 0.372 rpy=0.0 0.0 0.0
- added joint rear_axle_ground_to_luminar_front: type fixed, parent rear_axle_middle, child luminar_front, origin xyz=2.222 0.005 0.448 rpy=0.0 0.0 0.0
- added joint rear_axle_ground_to_luminar_left: type fixed, parent rear_axle_middle, child luminar_left, origin xyz=1.564 0.149 0.535 rpy=0 0 1.96349375
- added joint rear_axle_ground_to_luminar_right: type fixed, parent rear_axle_middle, child luminar_right, origin xyz=1.564 -0.153 0.535 rpy=0 0 -1.96349375
- added joint rear_axle_ground_to_radar_front: type fixed, parent rear_axle_middle, child radar_front, origin xyz=1.789 0.0 0.578 rpy=0.0 0.0 0.0
- added joint rear_axle_ground_to_radar_rear: type fixed, parent rear_axle_middle, child radar_rear, origin xyz=-0.752 0.0 0.107 rpy=0.0 0.0 3.14159
- added joint rear_axle_middle_proj_to_ground: type fixed, parent rear_axle_middle, child rear_axle_middle_ground, origin xyz=0.0 0.0 -0.306 rpy=0.0 0.0 0.0
- added joint rear_axle_middle_to_cog: type fixed, parent rear_axle_middle, child center_of_gravity, origin xyz=1.248156 0.0 -0.025 rpy=0.0 0.0 0.0
- added joint rear_axle_middle_to_front_axle_middle: type fixed, parent rear_axle_middle, child front_axle_middle, origin xyz=2.9718 0.0 -0.0055 rpy=0.0 0.0 0.0

Commit message: all cameras working with toggle

File: site/RacingSim/Sensors/av24.urdf (robot description, URDF)
Before this commit: robot AV24, 24 links, 23 joints
Links:
- removed link base_link
- removed link camera_front_roll_hoop
- removed link camera_front_stereo_left
- removed link camera_front_stereo_right
- removed link camera_rear_roll_hoop
- removed link front_axle_middle
- removed link gps_bottom_ant1
- removed link gps_bottom_imu
- removed link gps_spare
- removed link gps_spare_imu
- removed link gps_top_ant1
- removed link gps_top_imu
- removed link rear_axle_middle_ground
- added link camera_front_1
- added link camera_front_2
- added link camera_rear_left
- added link camera_rear_right
- added link gps_bottom_primary_antenna
- added link gps_bottom_secondary_antenna
- added link gps_top_primary_antenna
- added link gps_top_secondary_antenna
- added link radar_port
- added link radar_starboard
- added link vectornav
- added link vectornav_primary_antenna
- added link vectornav_secondary_antenna
Joints:
- removed joint base_link_to_rear_axle_middle
- removed joint gps_bottom_to_imu_bottom
- removed joint gps_spare_to_imu_spare
- removed joint gps_top_to_imu_top
- removed joint rear_axle_ground_to_camera_front_left
- removed joint rear_axle_ground_to_camera_front_right
- removed joint rear_axle_ground_to_camera_front_roll_hoop
- removed joint rear_axle_ground_to_camera_rear_roll_hoop
- removed joint rear_axle_ground_to_camera_stereo_left
- removed joint rear_axle_ground_to_camera_stereo_right
- removed joint rear_axle_ground_to_gps_bottom
- removed joint rear_axle_ground_to_gps_bottom_ant1
- removed joint rear_axle_ground_to_gps_spare
- removed joint rear_axle_ground_to_gps_top
- removed joint rear_axle_ground_to_gps_top_ant1
- removed joint rear_axle_ground_to_luminar_front
- removed joint rear_axle_ground_to_luminar_left
- removed joint rear_axle_ground_to_luminar_right
- removed joint rear_axle_ground_to_radar_front
- removed joint rear_axle_ground_to_radar_rear
- removed joint rear_axle_middle_proj_to_ground
- removed joint rear_axle_middle_to_cog
- removed joint rear_axle_middle_to_front_axle_middle
- added joint camera_front_1_joint: type fixed, parent rear_axle_middle, child camera_front_1, origin xyz=2.235 0.121 0.422
- added joint camera_front_2_joint: type fixed, parent rear_axle_middle, child camera_front_2, origin xyz=2.235 -0.121 0.422
- added joint camera_front_left_joint: type fixed, parent rear_axle_middle, child camera_front_left, origin xyz=2.184 0.171 0.422 rpy=0 0 0.9599310886
- added joint camera_front_right_joint: type fixed, parent rear_axle_middle, child camera_front_right, origin xyz=2.184 -0.171 0.422 rpy=0 0 -0.9599310886
- added joint camera_rear_left_joint: type fixed, parent rear_axle_middle, child camera_rear_left, origin xyz=1.473 0.140 0.543 rpy=0 0 2.2689280276
- added joint camera_rear_right_joint: type fixed, parent rear_axle_middle, child camera_rear_right, origin xyz=1.473 -0.140 0.543 rpy=0 0 -2.2689280276
- added joint gps_bottom_joint: type fixed, parent rear_axle_middle, child gps_bottom, origin xyz=1.636 0.075 -0.07427
- added joint gps_bottom_primary_antenna_joint: type fixed, parent gps_bottom, child gps_bottom_primary_antenna, origin xyz=0.419 -0.572 0.47876
- added joint gps_bottom_secondary_antenna_joint: type fixed, parent gps_bottom, child gps_bottom_secondary_antenna, origin xyz=-0.36449 0.07525 1.02668
- added joint gps_top_joint: type fixed, parent rear_axle_middle, child gps_top, origin xyz=1.636 -0.075 -0.07427
- added joint gps_top_primary_antenna_joint: type fixed, parent gps_top, child gps_top_primary_antenna, origin xyz=1.54 0.075 0.45940
- added joint gps_top_secondary_antenna_joint: type fixed, parent gps_top, child gps_top_secondary_antenna, origin xyz=0.41919 0.42225 0.45940
- added joint luminar_front_joint: type fixed, parent rear_axle_middle, child luminar_front, origin xyz=2.242 0 0.448
- added joint luminar_left_joint: type fixed, parent rear_axle_middle, child luminar_left, origin xyz=1.549 0.267 0.543 rpy=0 0 2.0943951024
- added joint luminar_right_joint: type fixed, parent rear_axle_middle, child luminar_right, origin xyz=1.549 -0.267 0.543 rpy=0 0 -2.0943951024
- added joint radar_front_joint: type fixed, parent rear_axle_middle, child radar_front, origin xyz=1.784 0.0 0.594
- added joint radar_port_joint: type fixed, parent rear_axle_middle, child radar_port, origin xyz=2.032 0.213 0.406 rpy=0 0 1.5707963267949
- added joint radar_starboard_joint: type fixed, parent rear_axle_middle, child radar_starboard, origin xyz=2.032 -0.213 0.406 rpy=0 0 -1.5707963267949
- added joint rear_axle_middle_joint: type fixed, parent center_of_gravity, child rear_axle_middle, origin xyz=-1.3206 0.030188 -0.23598
- added joint vectornav_joint: type fixed, parent rear_axle_middle, child vectornav, origin xyz=2.04486 0.118 0.49449
- added joint vectornav_primary_antenna_joint: type fixed, parent vectornav, child vectornav_primary_antenna, origin xyz=1.1 -0.118 -0.09
- added joint vectornav_secondary_antenna_joint: type fixed, parent vectornav, child vectornav_secondary_antenna, origin xyz=-0.80431 -0.118 0.45792
